File: electrical design/layer2/layer2.kicad_pcb (KiCad board)
At the start: 2 copper layers, 178 x 168.1 mm, 36 parts, among them J1 Conn_01x01_Female, J10 Conn_01x01_Female, J2 Conn_01x01_Female, J3 Conn_01x01_Female, J4 Conn_01x01_Female, J5 Conn_01x01_Female, J6 Conn_01x01_Female, J7 Conn_01x01_Female, J8 Conn_01x01_Female, J9 Conn_01x01_Female

Commit message: placed layer 2 mth
Parts:
- moved H4 20.0 mm to (182.5, 137.4)
- moved H3 19.5 mm to (182.5, 72.6)
- moved H8 15.6 mm to (27.5, 72.6)
- moved H7 14.8 mm to (27.5, 137.4)
- moved H6 13.9 mm to (59.6, 175.7)
- moved H5 12.6 mm to (150.4, 175.7)
- moved H17 9.06 mm to (102.0, 78.0)
- moved H23 8.63 mm to (102.0, 108.0)
- moved H18 8.14 mm to (102.0, 102.0)
- moved H21 8.06 mm to (108.0, 108.0)
- moved H19 8.02 mm to (108.0, 78.0)
- moved H20 7.52 mm to (108.0, 102.0)
- moved H14 7.19 mm to (137.9, 150.9)
- moved H12 7.05 mm to (155.9, 80.6)
- moved H22 7.02 mm to (108.0, 132.0)
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