File: electrical design/layer2/layer2.kicad_pcb (KiCad board)
At the start: 2 copper layers, 178 x 168.1 mm, 48 parts, among them J1 Conn_01x01_Female, J10 Conn_01x01_Female, J11 SH1.0 3P, J12 XH2.54 3P, J13 XT60-F, J14 XH2.54 2P, J15 XT60-F, J16 XT60-F, J17 SH1.0 2P, J18 Conn_01x01_Female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

Commit message: add ducc finishes and route unconnected l3 items
Other:
- board text added: "ducc."

Commit message: finalise pcbs for production
Parts:
- added R2: 0R, Resistor_SMD:R_2512_6332Metric, F.Cu at (87.0, 152.6)
- J13, J15: value XT60-F -> XT30UPB-F
- J16: value XT60-F -> XT30PW-F
Connections:
- J17 pad 1: GND -> Net-(J17-Pin_1)
- J17 pad 2: GND -> Net-(J17-Pin_1)
Routing:
- net GND: track 27.1 -> 40.7 mm, vias 1 -> 0
- net Net-(J17-Pin_1): track 0.00 -> 5.18 mm
- net +3V3: track 6.26 -> 5.56 mm
Changed lines of the file:
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@@
   (net 4 "+3V3")
   (net 5 "Net-(J12-Pin_3)")
+  (net 6 "Net-(J17-Pin_1)")
   (footprint "Connector_AMASS:AMASS_XT30UPB-F_1x02_P5.0mm_Vertical" (layer "F.Cu")
     (at 143.357043 164.747279 -57.3)
@@
         (effects (font (size 1 1) (thickness 0.15)))
     )
-    (fp_text value "XT60-F" (at 2.5 4 -57.3) (layer "F.Fab")
+    (fp_text value "XT30UPB-F" (at 2.5 4 -57.3) (layer "F.Fab")
         (effects (font (size 1 1) (thickness 0.15)))
     )
@@
       (stroke (width 0.1) (type solid)) (layer "F.Fab"))
     (pad "1" smd roundrect (at -0.5 -2 90) (size 0.6 1.55) (layers "F.Cu" "F.Paste" "F.Mask") (roundrect_rratio 0.25)
-      (net 2 "GND") (pinfunction "Pin_1") (pintype "passive"))
+      (net 6 "Net-(J17-Pin_1)") (pinfunction "Pin_1") (pintype "passive"))
     (pad "2" smd roundrect (at 0.5 -2 90) (size 0.6 1.55) (layers "F.Cu" "F.Paste" "F.Mask") (roundrect_rratio 0.25)
-      (net 2 "GND") (pinfunction "Pin_2") (pintype "passive"))
+      (net 6 "Net-(J17-Pin_1)") (pinfunction "Pin_2") (pintype "passive"))
     (pad "MP" smd roundrect (at -1.8 1.875 90) (size 1.2 1.8) (layers "F.Cu" "F.Paste" "F.Mask") (roundrect_rratio 0.2083333333))
     (pad "MP" smd roundrect (at 1.8 1.875 90) (size 1.2 1.8) (layers "F.Cu" "F.Paste" "F.Mask") (roundrect_rratio 0.2083333333))
@@
         (effects (font (size 1 1) (thickness 0.15)))
     )
-    (fp_text value "XT60-F" (at 2.5 4) (layer "F.Fab")
+    (fp_text value "XT30UPB-F" (at 2.5 4) (layer "F.Fab")
         (effects (font (size 1 1) (thickness 0.15)))
     )
@@
     )
   )
+  (footprint "Resistor_SMD:R_2512_6332Metric" (layer "F.Cu")
+    (at 87 152.6375 -90)
+    (descr "Resistor SMD 2512 (6332 Metric), square (rectangular) end terminal, IPC_7351 nominal, (Body size source: IPC-SM-782 page 72, https://www.pcb-3d.com/wordpress/wp-content/uploads/ipc-sm-782a_amendment_1_and_2.pdf), generated with kicad-footprint-generator")
+    (tags "resistor")
+    (property "Sheetfile" "layer2.kicad_sch")
+    (property "Sheetname" "")
+    (property "ki_description" "Resistor")
+    (property "ki_keywords" "R res resistor")
+    (attr smd)
+    (fp_text reference "R2" (at 0 -2.62 -90) (layer "F.SilkS")
+        (effects (font (size 1 1) (thickness 0.15)))
+    )
+    (fp_text value "0R" (at 0 2.62 -90) (layer "F.SilkS")
+        (effects (font (size 1 1) (thickness 0.15)))
+    )
+    (fp_text user "${REFERENCE}" (at 0 0 -90) (layer "F.Fab")
+        (effects (font (size 1 1) (thickness 0.15)))
+    )
+    (fp_line (start -2.177064 -1.71) (end 2.177064 -1.71)
+      (stroke (width 0.12) (type solid)) (layer "F.SilkS"))
+    (fp_line (start -2.177064 1.71) (end 2.177064 1.71)
+      (stroke (width 0.12) (type solid)) (layer "F.SilkS"))
+    (fp_line (start -3.82 -1.92) (end 3.82 -1.92)
+      (stroke (width 0.05) (type solid)) (layer "F.CrtYd"))
+    (fp_line (start -3.82 1.92) (end -3.82 -1.92)
+      (stroke (width 0.05) (type solid)) (layer "F.CrtYd"))
+    (fp_line (start 3.82 -1.92) (end 3.82 1.92)
+      (stroke (width 0.05) (type solid)) (layer "F.CrtYd"))
+    (fp_line (start 3.82 1.92) (end -3.82 1.92)
+      (stroke (width 0.05) (type solid)) (layer "F.CrtYd"))
+    (fp_line (start -3.15 -1.6) (end 3.15 -1.6)
+      (stroke (width 0.1) (type solid)) (layer "F.Fab"))
+    (fp_line (start -3.15 1.6) (end -3.15 -1.6)
+      (stroke (width 0.1) (type solid)) (layer "F.Fab"))
+    (fp_line (start 3.15 -1.6) (end 3.15 1.6)
+      (stroke (width 0.1) (type solid)) (layer "F.Fab"))
+    (fp_line (start 3.15 1.6) (end -3.15 1.6)
+      (stroke (width 0.1) (type solid)) (layer "F.Fab"))
+    (pad "1" smd roundrect (at -2.9625 0 270) (size 1.225 3.35) (layers "F.Cu" "F.Paste" "F.Mask") (roundrect_rratio 0.2040816327)
+      (net 6 "Net-(J17-Pin_1)") (pintype "passive"))
+    (pad "2" smd roundrect (at 2.9625 0 270) (size 1.225 3.35) (layers "F.Cu" "F.Paste" "F.Mask") (roundrect_rratio 0.2040816327)
+      (net 2 "GND") (pintype "passive"))
+    (model "${KICAD6_3DMODEL_DIR}/Resistor_SMD.3dshapes/R_2512_6332Metric.wrl"
+      (offset (xyz 0 0 0))
+      (scale (xyz 1 1 1))
+      (rotate (xyz 0 0 0))
+    )
+  )
   (footprint "MountingHole:MountingHole_2.2mm_M2_Pad" (layer "F.Cu")
     (at 63.306373 29.782705)
@@
     (property "ki_keywords" "mounting hole")
     (attr exclude_from_pos_files)
-    (fp_text reference "H33" (at 0 -3.2) (layer "F.SilkS") hide
+    (fp_text reference "H33" (at 0 -3.2) (layer "F.Fab")
         (effects (font (size 1 1) (thickness 0.15)))
     )
@@
         (effects (font (size 1 1) (thickness 0.15)))
     )
-    (fp_text user "${REFERENCE}" (at 0.3 0) (layer "F.Fab")
+    (fp_text user "${REFERENCE}" (at 0 0) (layer "F.Fab")
         (effects (font (size 1 1) (thickness 0.15)))
     )
@@
         (effects (font (size 1 1) (thickness 0.15)))
     )
-    (fp_text value "XT60-F" (at 2.5 3.5) (layer "F.Fab")
+    (fp_text value "XT30PW-F" (at 2.5 3.5) (layer "F.Fab")
         (effects (font (size 1 1) (thickness 0.15)))
     )
@@
     (property "ki_keywords" "mounting hole")
     (attr exclude_from_pos_files)
-    (fp_text reference "H34" (at 0 -3.2) (layer "F.SilkS") hide
+    (fp_text reference "H34" (at 0 -3.2) (layer "F.Fab")
         (effects (font (size 1 1) (thickness 0.15)))
     )
@@
         (effects (font (size 1 1) (thickness 0.15)))
     )
-    (fp_text user "${REFERENCE}" (at 0.3 0) (layer "F.Fab")
+    (fp_text user "${REFERENCE}" (at 0 0) (layer "F.Fab")
         (effects (font (size 1 1) (thickness 0.15)))
     )
@@
     (effects (font (size 0.8 0.8) (thickness 0.15) bold))
   )
-  (segment (start 87 144.5) (end 87 145.5) (width 0.25) (layer "F.Cu") (net 2))
-  (segment (start 78 166) (end 82 170) (width 0.25) (layer "F.Cu") (net 2))
-  (segment (start 78 165) (end 77 165) (width 0.25) (layer "F.Cu") (net 2))
-  (segment (start 76 166) (end 76 170) (width 0.25) (layer "F.Cu") (net 2))
-  (segment (start 81 175) (end 82 175) (width 0.25) (layer "F.Cu") (net 2))
-  (segment (start 82 171.25) (end 82 175) (width 0.25) (layer "F.Cu") (net 2))
-  (segment (start 82 170) (end 82 171.25) (width 0.25) (layer "F.Cu") (net 2))
-  (segment (start 76 170) (end 81 175) (width 0.25) (layer "F.Cu") (net 2))
-  (segment (start 87 145.5) (end 87 146.5) (width 0.25) (layer "F.Cu") (net 2))
-  (segment (start 77 165) (end 76 166) (width 0.25) (layer "F.Cu") (net 2))
-  (via (at 87 146.5) (size 0.8) (drill 0.4) (layers "F.Cu" "B.Cu") (net 2))
+  (segment (start 82 171.4) (end 82 175) (width 0.25) (layer "F.Cu") (net 2))
+  (segment (start 78 165) (end 78.8 165) (width 0.25) (layer "F.Cu") (net 2))
+  (segment (start 83.775 160.625) (end 83.775 173.225) (width 0.25) (layer "F.Cu") (net 2))
+  (segment (start 79.4 165.6) (end 79.4 167.6) (width 0.25) (layer "F.Cu") (net 2))
+  (segment (start 79.4 167.6) (end 82 170.2) (width 0.25) (layer "F.Cu") (net 2))
+  (segment (start 78.8 165) (end 79.4 165.6) (width 0.25) (layer "F.Cu") (net 2))
+  (segment (start 78 167.4) (end 82 171.4) (width 0.25) (layer "F.Cu") (net 2))
+  (segment (start 78 166) (end 78 167.4) (width 0.25) (layer "F.Cu") (net 2))
+  (segment (start 82 170.2) (end 82 171.4) (width 0.25) (layer "F.Cu") (net 2))
+  (segment (start 87 155.6) (end 87 157.4) (width 0.25) (layer "F.Cu") (net 2))
+  (segment (start 87 157.4) (end 83.775 160.625) (width 0.25) (layer "F.Cu") (net 2))
+  (segment (start 83.775 173.225) (end 82 175) (width 0.25) (layer "F.Cu") (net 2))
   (segment (start 78 164) (end 76.5 164) (width 0.25) (layer "F.Cu") (net 4))
   (segment (start 76.5 164) (end 76.25 164.25) (width 0.25) (layer "F.Cu") (net 4))
   (via (at 76.25 164.25) (size 0.8) (drill 0.4) (layers "F.Cu" "B.Cu") (net 4))
-  (segment (start 76.25 164.25) (end 75.75 164.75) (width 0.25) (layer "B.Cu") (net 4))
-  (segment (start 76.25 164.25) (end 75.75272 164.74728) (width 0.25) (layer "B.Cu") (net 4))
+  (segment (start 75.75 164.75) (end 76.25 164.25) (width 0.25) (layer "B.Cu") (net 4))
   (segment (start 75.75 164.75) (end 72.75 164.75) (width 0.25) (layer "B.Cu") (net 4))
   (segment (start 71.1 164.75) (end 66.645677 164.75) (width 0.25) (layer "B.Cu") (net 5))
   (segment (start 66.645677 164.75) (end 66.642957 164.74728) (width 0.25) (layer "B.Cu") (net 5))
+  (segment (start 87 144.5) (end 87 145.5) (width 0.25) (layer "F.Cu") (net 6))
+  (segment (start 87 145.5) (end 87 149.675) (width 0.25) (layer "F.Cu") (net 6))
   (zone (net 1) (net_name "+12V") (layer "F.Cu") (hatch edge 0.508)
     (connect_pads yes (clearance 0.508))
