File: electrical design/layer2/layer2.kicad_sch (KiCad schematic)
At the start: 48 parts, among them J1 Conn_01x01_Female, J1 XT60-F, J10 Conn_01x01_Female, J11 SH1.0 3P, J12 XH2.54 3P, J14 SH1.0 2P, J14 XH2.54 2P, J18 Conn_01x01_Female, J19 Conn_01x01_Female, J2 Conn_01x01_Female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

Commit message: finalise pcbs for production
Parts:
- added R2: 0R, Resistor_SMD:R_2512_6332Metric, symbol Device:R
- J1: value XT60-F -> XT30UPB-F
- J1: value XT60-F -> XT30PW-F
Connections:
- net GND: now also R2.2; no longer J14.1 (Pin_1), J14.2 (Pin_2)
- new net: J14.1 (Pin_1), J14.2 (Pin_2), R2.1
Changed lines of the file:
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@@
     (company "8076ducc Robotics Competition Team")
+  )
+  (junction (at 74.295 127.635) (diameter 0) (color 0 0 0 0)
+  )
+  (wire (pts (xy 74.295 127.635) (xy 74.295 130.175))
+    (stroke (width 0) (type default))
   )
   (label "BATT" (at 34.925 123.19 180) (fields_autoplaced)
@@
     )
   )
+  (symbol (lib_name "GND_1") (lib_id "power:GND") (at 81.915 127.635 90) (unit 1)
+    (in_bom yes) (on_board yes) (dnp no) (fields_autoplaced)
+    (property "Reference" "#PWR013" (at 88.265 127.635 0)
+      (effects (font (size 1.27 1.27)) hide)
+    )
+    (property "Value" "GND" (at 85.09 127.635 90)
+      (effects (font (size 1.27 1.27)) (justify right))
+    )
+    (property "Footprint" "" (at 81.915 127.635 0)
+      (effects (font (size 1.27 1.27)) hide)
+    )
+    (property "Datasheet" "" (at 81.915 127.635 0)
+      (effects (font (size 1.27 1.27)) hide)
+    )
+    (pin "1")
+    (instances
+      (project "layer2"
+        (path "/c8578fbc-a4a8-4ef3-83ea-12d29e2f2e36"
+          (reference "#PWR013") (unit 1)
+        )
+      )
+    )
+  )
   (symbol (lib_id "Connector:Conn_01x03_Pin") (at 20.955 82.55 0) (unit 1)
     (in_bom yes) (on_board yes) (dnp no) (fields_autoplaced)
@@
       (effects (font (size 1.27 1.27)))
     )
-    (property "Value" "XT60-F" (at 32.385 88.9 0)
+    (property "Value" "XT30UPB-F" (at 32.385 88.9 0)
       (effects (font (size 1.27 1.27)))
     )
@@
     )
   )
-  (symbol (lib_id "power:GND") (at 74.295 130.175 90) (unit 1)
-    (in_bom yes) (on_board yes) (dnp no) (fields_autoplaced)
-    (property "Reference" "#PWR014" (at 80.645 130.175 0)
-      (effects (font (size 1.27 1.27)) hide)
-    )
-    (property "Value" "GND" (at 78.105 130.175 90)
-      (effects (font (size 1.27 1.27)) (justify right))
-    )
-    (property "Footprint" "" (at 74.295 130.175 0)
-      (effects (font (size 1.27 1.27)) hide)
-    )
-    (property "Datasheet" "" (at 74.295 130.175 0)
-      (effects (font (size 1.27 1.27)) hide)
-    )
-    (pin "1")
-    (instances
-      (project "layer2"
-        (path "/c8578fbc-a4a8-4ef3-83ea-12d29e2f2e36"
-          (reference "#PWR014") (unit 1)
-        )
-      )
-    )
-  )
   (symbol (lib_id "power:GND") (at 33.02 66.04 270) (unit 1)
     (in_bom yes) (on_board yes) (dnp no) (fields_autoplaced)
@@
   (symbol (lib_id "Connector:Conn_01x02_Female") (at 69.215 120.015 180) (unit 1)
     (in_bom yes) (on_board yes) (dnp no) (fields_autoplaced)
-    (property "Reference" "J1" (at 69.85 112.395 0)
-      (effects (font (size 1.27 1.27)))
-    )
-    (property "Value" "XT60-F" (at 69.85 114.935 0)
+    (property "Reference" "J1" (at 69.85 111.76 0)
+      (effects (font (size 1.27 1.27)))
+    )
+    (property "Value" "XT30PW-F" (at 69.85 114.3 0)
       (effects (font (size 1.27 1.27)))
     )
@@
     )
   )
+  (symbol (lib_id "Device:R") (at 78.105 127.635 90) (unit 1)
+    (in_bom yes) (on_board yes) (dnp no) (fields_autoplaced)
+    (property "Reference" "R2" (at 78.105 121.92 90)
+      (effects (font (size 1.27 1.27)))
+    )
+    (property "Value" "0R" (at 78.105 124.46 90)
+      (effects (font (size 1.27 1.27)))
+    )
+    (property "Footprint" "Resistor_SMD:R_2512_6332Metric" (at 78.105 129.413 90)
+      (effects (font (size 1.27 1.27)) hide)
+    )
+    (property "Datasheet" "~" (at 78.105 127.635 0)
+      (effects (font (size 1.27 1.27)) hide)
+    )
+    (pin "2")
+    (pin "1")
+    (instances
+      (project "layer2"
+        (path "/c8578fbc-a4a8-4ef3-83ea-12d29e2f2e36"
+          (reference "R2") (unit 1)
+        )
+      )
+    )
+  )
   (symbol (lib_id "Mechanical:MountingHole") (at 80.01 55.88 0) (unit 1)
     (in_bom yes) (on_board yes) (dnp no) (fields_autoplaced)
@@
       (effects (font (size 1.27 1.27)))
     )
-    (property "Value" "XT60-F" (at 69.85 104.14 0)
+    (property "Value" "XT30UPB-F" (at 69.85 104.14 0)
       (effects (font (size 1.27 1.27)))
     )
@@
         )
       )
-    )
-  )
-  (symbol (lib_id "power:GND") (at 74.295 127.635 90) (unit 1)
-    (in_bom yes) (on_board yes) (dnp no) (fields_autoplaced)
-    (property "Reference" "#PWR013" (at 80.645 127.635 0)
-      (effects (font (size 1.27 1.27)) hide)
-    )
-    (property "Value" "GND" (at 77.47 127.635 90)
-      (effects (font (size 1.27 1.27)) (justify right))
-    )
-    (property "Footprint" "" (at 74.295 127.635 0)
-      (effects (font (size 1.27 1.27)) hide)
-    )
-    (property "Datasheet" "" (at 74.295 127.635 0)
-      (effects (font (size 1.27 1.27)) hide)
-    )
-    (pin "1")
-    (instances
-      (project "layer2"
-        (path "/c8578fbc-a4a8-4ef3-83ea-12d29e2f2e36"
-          (reference "#PWR013") (unit 1)
-        )
-      )
