File: electrical design/layer1/layer1.kicad_pcb (KiCad board)
At the start: 2 copper layers, 178 x 168.1 mm, 225 parts, among them J1 XT30-F, J10 Conn_01x02_Pin, J11 Conn_01x01_Socket, J12 Conn_01x01_Socket, J13 Conn_01x05_Pin, J14 Conn_01x02_Pin, J2 Conn_01x01_Socket, J3 Conn_01x01_Socket, J4 XT30PW-F, J5 Conn_01x01_Socket, J6 Conn_01x01_Socket, J7 Conn_01x01_Socket, J8 Conn_01x01_Socket, J9 Conn_01x02_Pin, Q1 MOSFET-NCH-FQP30N06L, Q2 MOSFET-NCH-AO3404A, SW1 SW_SPDT, U1 CD74HC4067SM, U2 CD74HC4067SM, U3 MOUDLE-SEEEDUINO-XIAO-ESP32C3

Commit message: add jlc order number silkscreen
Other:
- board text added: "JLCJLCJLCJLC"
Changed lines of the file:
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@@
     (pad "2" smd roundrect (at 0.5 1.325) (size 0.6 1.55) (layers "F.Cu" "F.Paste" "F.Mask") (roundrect_rratio 0.25)
       (net 123 "GNDD") (pinfunction "Pin_2") (pintype "passive"))
-    (pad "MP" smd roundrect (at -1.8 -1.2) (size 1.2 1.8) (layers "F.Cu" "F.Paste" "F.Mask") (roundrect_rratio 0.208333))
-    (pad "MP" smd roundrect (at 1.8 -1.2) (size 1.2 1.8) (layers "F.Cu" "F.Paste" "F.Mask") (roundrect_rratio 0.208333))
+    (pad "MP" smd roundrect (at -1.8 -1.2) (size 1.2 1.8) (layers "F.Cu" "F.Paste" "F.Mask") (roundrect_rratio 0.2083333333))
+    (pad "MP" smd roundrect (at 1.8 -1.2) (size 1.2 1.8) (layers "F.Cu" "F.Paste" "F.Mask") (roundrect_rratio 0.2083333333))
     (model "${KICAD7_3DMODEL_DIR}/Connector_JST.3dshapes/JST_SH_BM02B-SRSS-TB_1x02-1MP_P1.00mm_Vertical.step"
       (offset (xyz 0 1 0))
@@
     (effects (font (size 1.5 1.5) (thickness 0.3)))
   )
+  (gr_text "JLCJLCJLCJLC" (at 119 146) (layer "F.SilkS")
+    (effects (font (size 1 1) (thickness 0.2) bold))
+  )
   (gr_text "ON" (at 45.75 123) (layer "F.SilkS")

Commit message: add ducc finishes and route unconnected l3 items
Parts:
- added G***: LOGO, LOGO, F.Cu at (105.0, 105.0)
- added G***: LOGO, LOGO, F.Cu at (105.0, 97.0)
Routing:
- net /S1: track 111.2 -> 110.5 mm

Commit message: finalise pcbs for production
Parts:
- added J15: Conn_01x01_Socket, Connector_Wire:SolderWirePad_1x01_SMD_1x2mm, F.Cu at (111.8, 169.6)
- J14: value Conn_01x02_Pin -> SH1.0 3P; footprint Connector_JST:JST_SH_BM02B-SRSS-TB_1x02-1MP_P1.00mm_Vertical -> Connector_JST:JST_SH_BM03B-SRSS-TB_1x03-1MP_P1.00mm_Vertical
- R1, R10, R11, R12, R13, R14, R15, R16, R17, R18, R19, R2, R20, R21, R22, R23, R24, R25, R26, R27, R28, R29, R3, R30, R31, R32, R4, R5, R6, R7, R8, R9: value 0.39 -> 0R39
- moved J4 5.00 mm to (137.2, 174.0), turned to -90 degrees
- moved J13 1.50 mm to (177.7, 119.6)
- moved U3 1.50 mm to (177.8, 105.0)
Routing:
- net +48V: track 36.7 -> 34.6 mm
- net GNDD: track 120.3 -> 118.7 mm
- net /SOLENOIDON: track 96.3 -> 94.8 mm
- net /S3: track 102.2 -> 100.7 mm
- net /S2: track 106.6 -> 105.1 mm
- net /S1: track 110.5 -> 109.0 mm
- net /S0: track 114.3 -> 112.8 mm
- net /MUX2OUT: track 49.0 -> 47.5 mm
- net /MUX1OUT: track 125.8 -> 124.3 mm
- net /BALL: track 99.0 -> 98.4 mm
Other:
- board text added: "LED"

Commit message: correct led inductor value
Parts:
- J13: value Conn_01x05_Pin -> SH1.0 5P
- L1, L10, L11, L12, L13, L14, L15, L16, L17, L18, L19, L2, L20, L21, L22, L23, L24, L25, L26, L27, L28, L29, L3, L30, L31, L32, L4, L5, L6, L7, L8, L9: value 10mA -> 10µH
Changed lines of the file:
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@@
         (effects (font (size 1 1) (thickness 0.15)))
     )
-    (fp_text value "Conn_01x05_Pin" (at 0 3.3) (layer "F.Fab")
+    (fp_text value "SH1.0 5P" (at 0 3.3) (layer "F.Fab")
         (effects (font (size 1 1) (thickness 0.15)))
     )
@@
         (effects (font (size 1 1) (thickness 0.15)) (justify mirror))
     )
-    (fp_text value "10mA" (at 4.190476 0 101.25) (layer "B.SilkS") hide
+    (fp_text value "10µH" (at 4.190476 0 101.25) (layer "B.SilkS") hide
         (effects (font (size 1 1) (thickness 0.15)) (justify mirror))
     )
@@
         (effects (font (size 1 1) (thickness 0.15)) (justify mirror))
     )
-    (fp_text value "10mA" (at 4.190476 0 112.5) (layer "B.SilkS") hide
+    (fp_text value "10µH" (at 4.190476 0 112.5) (layer "B.SilkS") hide
         (effects (font (size 1 1) (thickness 0.15)) (justify mirror))
     )
@@
         (effects (font (size 1 1) (thickness 0.15)) (justify mirror))
     )
-    (fp_text value "10mA" (at 4.190476 0 146.25) (layer "B.SilkS") hide
+    (fp_text value "10µH" (at 4.190476 0 146.25) (layer "B.SilkS") hide
         (effects (font (size 1 1) (thickness 0.15)) (justify mirror))
     )
@@
         (effects (font (size 1 1) (thickness 0.15)) (justify mirror))
     )
-    (fp_text value "10mA" (at 4.190476 0 45) (layer "B.SilkS") hide
+    (fp_text value "10µH" (at 4.190476 0 45) (layer "B.SilkS") hide
         (effects (font (size 1 1) (thickness 0.15)) (justify mirror))
     )
@@
         (effects (font (size 1 1) (thickness 0.15)) (justify mirror))
     )
-    (fp_text value "10mA" (at 4.190476 0 33.75) (layer "B.SilkS") hide
+    (fp_text value "10µH" (at 4.190476 0 33.75) (layer "B.SilkS") hide
         (effects (font (size 1 1) (thickness 0.15)) (justify mirror))
     )
@@
         (effects (font (size 1 1) (thickness 0.15)) (justify mirror))
     )
-    (fp_text value "10mA" (at 4.190476 0 168.75) (layer "B.SilkS") hide
+    (fp_text value "10µH" (at 4.190476 0 168.75) (layer "B.SilkS") hide
         (effects (font (size 1 1) (thickness 0.15)) (justify mirror))
     )
@@
         (effects (font (size 1 1) (thickness 0.15)) (justify mirror))
     )
-    (fp_text value "10mA" (at 4.190476 0 157.5) (layer "B.SilkS") hide
+    (fp_text value "10µH" (at 4.190476 0 157.5) (layer "B.SilkS") hide
         (effects (font (size 1 1) (thickness 0.15)) (justify mirror))
     )
@@
         (effects (font (size 1 1) (thickness 0.15)) (justify mirror))
     )
-    (fp_text value "10mA" (at 4.190476 0 168.75) (layer "B.SilkS") hide
+    (fp_text value "10µH" (at 4.190476 0 168.75) (layer "B.SilkS") hide
         (effects (font (size 1 1) (thickness 0.15)) (justify mirror))
     )
@@
         (effects (font (size 1 1) (thickness 0.15)) (justify mirror))
     )
-    (fp_text value "10mA" (at 4.190476 0 135) (layer "B.SilkS") hide
+    (fp_text value "10µH" (at 4.190476 0 135) (layer "B.SilkS") hide
         (effects (font (size 1 1) (thickness 0.15)) (justify mirror))
     )
@@
         (effects (font (size 1 1) (thickness 0.15)) (justify mirror))
     )
-    (fp_text value "10mA" (at 4.190476 0 90) (layer "B.SilkS") hide
+    (fp_text value "10µH" (at 4.190476 0 90) (layer "B.SilkS") hide
         (effects (font (size 1 1) (thickness 0.15)) (justify mirror))
     )
@@
         (effects (font (size 1 1) (thickness 0.15)) (justify mirror))
     )
-    (fp_text value "10mA" (at 4.190476 0 90) (layer "B.SilkS") hide
+    (fp_text value "10µH" (at 4.190476 0 90) (layer "B.SilkS") hide
         (effects (font (size 1 1) (thickness 0.15)) (justify mirror))
     )
@@
         (effects (font (size 1 1) (thickness 0.15)) (justify mirror))
     )
-    (fp_text value "10mA" (at 4.190476 0 33.75) (layer "B.SilkS") hide
+    (fp_text value "10µH" (at 4.190476 0 33.75) (layer "B.SilkS") hide
         (effects (font (size 1 1) (thickness 0.15)) (justify mirror))
     )
@@
         (effects (font (size 1 1) (thickness 0.15)) (justify mirror))
     )
-    (fp_text value "10mA" (at 4.190476 0 123.75) (layer "B.SilkS") hide
+    (fp_text value "10µH" (at 4.190476 0 123.75) (layer "B.SilkS") hide
         (effects (font (size 1 1) (thickness 0.15)) (justify mirror))
     )
@@
         (effects (font (size 1 1) (thickness 0.15)) (justify mirror))
     )
-    (fp_text value "10mA" (at 4.190476 0 56.25) (layer "B.SilkS") hide
+    (fp_text value "10µH" (at 4.190476 0 56.25) (layer "B.SilkS") hide
         (effects (font (size 1 1) (thickness 0.15)) (justify mirror))
     )
@@
         (effects (font (size 1 1) (thickness 0.15)) (justify mirror))
     )
-    (fp_text value "10mA" (at 4.190476 0 123.75) (layer "B.SilkS") hide
+    (fp_text value "10µH" (at 4.190476 0 123.75) (layer "B.SilkS") hide
         (effects (font (size 1 1) (thickness 0.15)) (justify mirror))
     )
@@
         (effects (font (size 1 1) (thickness 0.15)) (justify mirror))
     )
-    (fp_text value "10mA" (at 4.190476 0 67.5) (layer "B.SilkS") hide
+    (fp_text value "10µH" (at 4.190476 0 67.5) (layer "B.SilkS") hide
         (effects (font (size 1 1) (thickness 0.15)) (justify mirror))
     )
@@
         (effects (font (size 1 1) (thickness 0.15)) (justify mirror))
     )
-    (fp_text value "10mA" (at 4.190476 0 101.25) (layer "B.SilkS") hide
+    (fp_text value "10µH" (at 4.190476 0 101.25) (layer "B.SilkS") hide
         (effects (font (size 1 1) (thickness 0.15)) (justify mirror))
     )
@@
         (effects (font (size 1 1) (thickness 0.15)) (justify mirror))
     )
-    (fp_text value "10mA" (at 4.190476 0 11.25) (layer "B.SilkS") hide
+    (fp_text value "10µH" (at 4.190476 0 11.25) (layer "B.SilkS") hide
         (effects (font (size 1 1) (thickness 0.15)) (justify mirror))
     )
@@
         (effects (font (size 1 1) (thickness 0.15)) (justify mirror))
     )
-    (fp_text value "10mA" (at 4.190476 0 45) (layer "B.SilkS") hide
+    (fp_text value "10µH" (at 4.190476 0 45) (layer "B.SilkS") hide
         (effects (font (size 1 1) (thickness 0.15)) (justify mirror))
     )
@@
         (effects (font (size 1 1) (thickness 0.15)) (justify mirror))
     )
-    (fp_text value "10mA" (at 4.190476 0 22.5) (layer "B.SilkS") hide
+    (fp_text value "10µH" (at 4.190476 0 22.5) (layer "B.SilkS") hide
         (effects (font (size 1 1) (thickness 0.15)) (justify mirror))
     )
@@
         (effects (font (size 1 1) (thickness 0.15)) (justify mirror))
     )
-    (fp_text value "10mA" (at 4.190476 0 11.25) (layer "B.SilkS") hide
+    (fp_text value "10µH" (at 4.190476 0 11.25) (layer "B.SilkS") hide
         (effects (font (size 1 1) (thickness 0.15)) (justify mirror))
     )
@@
         (effects (font (size 1 1) (thickness 0.15)) (justify mirror))
     )
-    (fp_text value "10mA" (at 4.190476 0 78.75) (layer "B.SilkS") hide
+    (fp_text value "10µH" (at 4.190476 0 78.75) (layer "B.SilkS") hide
         (effects (font (size 1 1) (thickness 0.15)) (justify mirror))
     )
@@
         (effects (font (size 1 1) (thickness 0.15)) (justify mirror))
     )
-    (fp_text value "10mA" (at 4.190476 0 146.25) (layer "B.SilkS") hide
+    (fp_text value "10µH" (at 4.190476 0 146.25) (layer "B.SilkS") hide
         (effects (font (size 1 1) (thickness 0.15)) (justify mirror))
     )
@@
         (effects (font (size 1 1) (thickness 0.15)) (justify mirror))
     )
-    (fp_text value "10mA" (at 4.190476 0 157.5) (layer "B.SilkS") hide
+    (fp_text value "10µH" (at 4.190476 0 157.5) (layer "B.SilkS") hide
         (effects (font (size 1 1) (thickness 0.15)) (justify mirror))
     )
@@
         (effects (font (size 1 1) (thickness 0.15)) (justify mirror))
     )
-    (fp_text value "10mA" (at 4.190476 0 56.25) (layer "B.SilkS") hide
+    (fp_text value "10µH" (at 4.190476 0 56.25) (layer "B.SilkS") hide
         (effects (font (size 1 1) (thickness 0.15)) (justify mirror))
     )
@@
         (effects (font (size 1 1) (thickness 0.15)) (justify mirror))
     )
-    (fp_text value "10mA" (at 4.190476 0 67.5) (layer "B.SilkS") hide
+    (fp_text value "10µH" (at 4.190476 0 67.5) (layer "B.SilkS") hide
         (effects (font (size 1 1) (thickness 0.15)) (justify mirror))
     )
@@
         (effects (font (size 1 1) (thickness 0.15)) (justify mirror))
     )
-    (fp_text value "10mA" (at 4.190476 0 22.5) (layer "B.SilkS") hide
+    (fp_text value "10µH" (at 4.190476 0 22.5) (layer "B.SilkS") hide
         (effects (font (size 1 1) (thickness 0.15)) (justify mirror))
     )
@@
         (effects (font (size 1 1) (thickness 0.15)) (justify mirror))
     )
-    (fp_text value "10mA" (at 4.190476 0 112.5) (layer "B.SilkS") hide
+    (fp_text value "10µH" (at 4.190476 0 112.5) (layer "B.SilkS") hide
         (effects (font (size 1 1) (thickness 0.15)) (justify mirror))
     )
@@
         (effects (font (size 1 1) (thickness 0.15)) (justify mirror))
     )
-    (fp_text value "10mA" (at 4.190476 0 78.75) (layer "B.SilkS") hide
+    (fp_text value "10µH" (at 4.190476 0 78.75) (layer "B.SilkS") hide
         (effects (font (size 1 1) (thickness 0.15)) (justify mirror))
     )
@@
         (effects (font (size 1 1) (thickness 0.15)) (justify mirror))
     )
-    (fp_text value "10mA" (at 4.190476 0 135) (layer "B.SilkS") hide
+    (fp_text value "10µH" (at 4.190476 0 135) (layer "B.SilkS") hide
         (effects (font (size 1 1) (thickness 0.15)) (justify mirror))
     )
@@
         (effects (font (size 1 1) (thickness 0.15)) (justify mirror))
     )
-    (fp_text value "10mA" (at 4.190476 0) (layer "B.SilkS") hide
+    (fp_text value "10µH" (at 4.190476 0) (layer "B.SilkS") hide
         (effects (font (size 1 1) (thickness 0.15)) (justify mirror))
     )
@@
         (effects (font (size 1 1) (thickness 0.15)) (justify mirror))
     )
-    (fp_text value "10mA" (at 4.190476 0) (layer "B.SilkS") hide
+    (fp_text value "10µH" (at 4.190476 0) (layer "B.SilkS") hide
         (effects (font (size 1 1) (thickness 0.15)) (justify mirror))
     )
