File: lightweight/layer1/layer1.kicad_pcb (KiCad board)
At the start: 2 copper layers, 208 x 198.4 mm, 228 parts, among them J1 XT30-F, J10 Conn_01x02_Pin, J11 Conn_01x01_Socket, J12 Conn_01x01_Socket, J13 SH1.0 5P, J14 SH1.0 3P, J15 Conn_01x01_Socket, J2 Conn_01x01_Socket, J3 Conn_01x01_Socket, J4 XT30PW-F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

Commit message: added layer 2
Parts:
- moved R40 45.4 mm to (146.2, 173.4)
- moved Q2 36.3 mm to (144.7, 176.9), turned to 180 degrees
- moved J4 23.3 mm to (137.7, 178.8)
- moved Q1 16.7 mm to (136.5, 172.5), turned to 0 degrees
Routing:
- net Net-(D2-A): track 5.44 -> 35.6 mm, vias 0 -> 1
- net /SOLENOIDON: track 107.6 -> 79.7 mm
- net Net-(Q1-S): track 17.7 -> 39.7 mm, vias 0 -> 1
- net +48V: track 89.2 -> 107.1 mm
- net Net-(Q1-G): track 7.33 -> 22.4 mm, vias 0 -> 2
