File: lightweight/layer2/layer2.kicad_pcb (KiCad board)
At the start: 2 copper layers, 208 x 198.4 mm, 49 parts, among them J1 Conn_01x01_Female, J10 Conn_01x01_Female, J11 SH1.0 3P, J12 XH2.54 3P, J13 XT30UPB-F, J14 XH2.54 2P, J15 XT30UPB-F, J16 XT30PW-F, J17 SH1.0 2P, J18 Conn_01x01_Female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

Commit message: update lw pcbs
Parts:
- removed J12: XH2.54 3P, Connector_JST:JST_XH_B3B-XH-A_1x03_P2.50mm_Vertical
- removed J13: XT30UPB-F, Connector_AMASS:AMASS_XT30UPB-F_1x02_P5.0mm_Vertical
- removed R1: 10k, Resistor_SMD:R_0603_1608Metric
Routing:
- net +3V3: track 5.56 -> 0.00 mm, vias 1 -> 0
- net Net-(J12-Pin_3): track 4.46 -> 0.00 mm
