File: lightweight/layer2/layer2.kicad_sch (KiCad schematic)
At the start: 49 parts, among them J1 Conn_01x01_Female, J1 XT30PW-F, J1 XT30UPB-F, J10 Conn_01x01_Female, J11 SH1.0 3P, J12 XH2.54 3P, J14 SH1.0 2P, J14 XH2.54 2P, J18 Conn_01x01_Female, J19 Conn_01x01_Female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

Commit message: update lw pcbs
Parts:
- removed J1: XT30UPB-F, Connector_AMASS:AMASS_XT30UPB-F_1x02_P5.0mm_Vertical, symbol Connector:Conn_01x02_Female
- removed J12: XH2.54 3P, Connector_JST:JST_XH_B3B-XH-A_1x03_P2.50mm_Vertical, symbol Connector:Conn_01x03_Pin
- removed R1: 10k, Resistor_SMD:R_0603_1608Metric, symbol Device:R
