File: lightweight/layer3/layer3.kicad_sch (KiCad schematic)
At the start: 25 parts, among them J13 SH1.0 5P, J14 SH1.0 2P, J2 SH1.0 5P, J8 COMPASS, SW1 SW_SPDT, U1 TEENSY 4.0, U2 MOUDLE-SEEEDUINO-XIAO-ESP32C3, U4 74LVC2G04, U5 74LVC2G04, U6 74LVC2G04

Commit message: update lw pcbs
Parts:
- removed H5, H6: MountingHole, MountingHole:MountingHole_3.2mm_M3_Pad, symbol Mechanical:MountingHole
- removed J8: COMPASS, Connector_JST:JST_SH_BM04B-SRSS-TB_1x04-1MP_P1.00mm_Vertical, symbol Connector:Conn_01x04_Pin
- removed R6, R7: R, Resistor_SMD:R_0603_1608Metric, symbol Device:R
- added J5: Conn_01x16_Socket, symbol Connector:Conn_01x16_Socket
Connections:
- net SCL is gone; now on net IMUSCL: U?.JP1_4 (SCL)
- net SDA is gone; now on net IMUSDA: U?.JP1_5 (SDA)
- net +5V: now also J5.10 (Pin_10)
- net CAMRX: now also J5.1 (Pin_1)
- net CAMTX: now also J5.2 (Pin_2)
- net GND: now also J5.9 (Pin_9)
