File: lightweight/electrical design/layer2/layer2.kicad_sch (KiCad schematic)
At the start: 46 parts, among them J1 Conn_01x01_Female, J1 XT30PW-F, J1 XT30UPB-F, J10 Conn_01x01_Female, J11 SH1.0 3P, J14 SH1.0 2P, J14 XH2.54 2P, J18 Conn_01x01_Female, J19 Conn_01x01_Female, J2 Conn_01x01_Female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

Commit message: update lw pcbs
Parts:
- added H27, H28, H29, H30: MountingHole, MountingHole:MountingHole_3.2mm_M3_Pad, symbol Mechanical:MountingHole
Changed lines of the file:
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@@
+    )
+  )
+  (symbol (lib_id "Mechanical:MountingHole") (at 121.92 77.47 0) (unit 1)
+    (in_bom yes) (on_board yes) (dnp no)
+    (property "Reference" "H27" (at 124.968 76.1999 0)
+      (effects (font (size 1.27 1.27)) (justify left))
+    )
+    (property "Value" "MountingHole" (at 124.968 78.7399 0)
+      (effects (font (size 1.27 1.27)) (justify left))
+    )
+    (property "Footprint" "MountingHole:MountingHole_3.2mm_M3_Pad" (at 121.92 77.47 0)
+      (effects (font (size 1.27 1.27)) hide)
+    )
+    (property "Datasheet" "~" (at 121.92 77.47 0)
+      (effects (font (size 1.27 1.27)) hide)
+    )
+    (instances
+      (project "layer2"
+        (path "/c8578fbc-a4a8-4ef3-83ea-12d29e2f2e36"
+          (reference "H27") (unit 1)
+        )
+      )
     )
   )
@@
         (path "/c8578fbc-a4a8-4ef3-83ea-12d29e2f2e36"
           (reference "H12") (unit 1)
+        )
+      )
+    )
+  )
+  (symbol (lib_id "Mechanical:MountingHole") (at 121.92 82.55 0) (unit 1)
+    (in_bom yes) (on_board yes) (dnp no)
+    (property "Reference" "H28" (at 124.968 81.2799 0)
+      (effects (font (size 1.27 1.27)) (justify left))
+    )
+    (property "Value" "MountingHole" (at 124.968 83.8199 0)
+      (effects (font (size 1.27 1.27)) (justify left))
+    )
+    (property "Footprint" "MountingHole:MountingHole_3.2mm_M3_Pad" (at 121.92 82.55 0)
+      (effects (font (size 1.27 1.27)) hide)
+    )
+    (property "Datasheet" "~" (at 121.92 82.55 0)
+      (effects (font (size 1.27 1.27)) hide)
+    )
+    (instances
+      (project "layer2"
+        (path "/c8578fbc-a4a8-4ef3-83ea-12d29e2f2e36"
+          (reference "H28") (unit 1)
         )
       )
@@
     )
   )
+  (symbol (lib_id "Mechanical:MountingHole") (at 121.92 93.345 0) (unit 1)
+    (in_bom yes) (on_board yes) (dnp no)
+    (property "Reference" "H30" (at 124.968 92.0749 0)
+      (effects (font (size 1.27 1.27)) (justify left))
+    )
+    (property "Value" "MountingHole" (at 124.968 94.6149 0)
+      (effects (font (size 1.27 1.27)) (justify left))
+    )
+    (property "Footprint" "MountingHole:MountingHole_3.2mm_M3_Pad" (at 121.92 93.345 0)
+      (effects (font (size 1.27 1.27)) hide)
+    )
+    (property "Datasheet" "~" (at 121.92 93.345 0)
+      (effects (font (size 1.27 1.27)) hide)
+    )
+    (instances
+      (project "layer2"
+        (path "/c8578fbc-a4a8-4ef3-83ea-12d29e2f2e36"
+          (reference "H30") (unit 1)
+        )
+      )
+    )
+  )
   (symbol (lib_id "power:+12V") (at 33.02 35.56 90) (unit 1)
     (in_bom yes) (on_board yes) (dnp no) (fields_autoplaced)
@@
         )
       )
+    )
+  )
+  (symbol (lib_id "Mechanical:MountingHole") (at 121.92 88.265 0) (unit 1)
+    (in_bom yes) (on_board yes) (dnp no)
+    (property "Reference" "H29" (at 124.968 86.9949 0)
+      (effects (font (size 1.27 1.27)) (justify left))
+    )
+    (property "Value" "MountingHole" (at 124.968 89.5349 0)
+      (effects (font (size 1.27 1.27)) (justify left))
+    )
+    (property "Footprint" "MountingHole:MountingHole_3.2mm_M3_Pad" (at 121.92 88.265 0)
+      (effects (font (size 1.27 1.27)) hide)
+    )
+    (property "Datasheet" "~" (at 121.92 88.265 0)
+      (effects (font (size 1.27 1.27)) hide)
+    )
+    (instances
+      (project "layer2"
+        (path "/c8578fbc-a4a8-4ef3-83ea-12d29e2f2e36"
+          (reference "H29") (unit 1)
+        )
+      )
