File: lightweight/electrical design/layer2/layer2.kicad_pcb (KiCad board)
At the start: 2 copper layers, 208 x 198.4 mm, 46 parts, among them J1 Conn_01x01_Female, J10 Conn_01x01_Female, J11 SH1.0 3P, J14 XH2.54 2P, J15 XT30UPB-F, J16 XT30PW-F, J17 SH1.0 2P, J18 Conn_01x01_Female, J19 Conn_01x01_Female, J2 Conn_01x01_Female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

Commit message: update lw pcbs
Parts:
- added H27: MountingHole, MountingHole:MountingHole_3.2mm_M3_Pad, F.Cu at (89.0, 46.6)
- added H28: MountingHole, MountingHole:MountingHole_3.2mm_M3_Pad, F.Cu at (121.0, 46.6)
- added H29: MountingHole, MountingHole:MountingHole_3.2mm_M3_Pad, F.Cu at (89.0, 66.6)
- added H30: MountingHole, MountingHole:MountingHole_3.2mm_M3_Pad, F.Cu at (121.0, 66.6)
Other:
- outline, holes or cut-outs redrawn

Commit message: add lw pcb files
Parts:
- moved H1 28.3 mm to (67.8, 44.5)
- moved H12 28.3 mm to (187.4, 91.2)
- moved H13 28.3 mm to (187.4, 159.2)
- moved H14 28.3 mm to (169.4, 180.6)
- moved H16 28.3 mm to (62.6, 159.2)
- moved H17 28.3 mm to (122.0, 98.0)
- moved H18 28.3 mm to (122.0, 122.0)
- moved H19 28.3 mm to (128.0, 98.0)
- moved H2 28.3 mm to (182.2, 44.5)
- moved H20 28.3 mm to (128.0, 122.0)
- moved H21 28.3 mm to (128.0, 128.0)
- moved H22 28.3 mm to (128.0, 152.0)
- moved H23 28.3 mm to (122.0, 128.0)
- moved H24 28.3 mm to (122.0, 152.0)
- moved H25 28.3 mm to (98.0, 167.1)
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