File: lightweight/electrical design/layer3/layer3.kicad_pcb (KiCad board)
At the start: 2 copper layers, 189.7 x 105 mm, 60 parts, among them J1 SH1.0 5P, J10 SH1.0 2P, J11 SH1.0 5P, J2 SH1.0 5P, J3 SH1.0 5P, J5 Conn_01x16_Socket, J6 SH1.0 Female, SW1 SW_SPDT, SW5 SW_Push, U1 TEENSY 4.0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

Commit message: updater layer 3
Parts:
- J1, J10, J2, J3, locked: moved to B.Cu
- turned J1 to 0 degrees
- turned J10 to 180 degrees
- turned J2 to 0 degrees
- turned J3 to 180 degrees
- turned locked to 180 degrees
Routing:
- net /CAMTX: track 0.00 -> 73.0 mm, vias 0 -> 8
- net /CAMRX: track 0.00 -> 58.1 mm, vias 0 -> 4
- net /BTRX: track 0.00 -> 53.3 mm, vias 0 -> 2
- net +5V: track 92.1 -> 143.4 mm, vias 4 -> 8
- net GNDD: track 190.8 -> 144.5 mm, vias 21 -> 15
- net +3V3: track 493.2 -> 532.0 mm, vias 5 -> 11
- net /BTTX: track 0.00 -> 33.6 mm, vias 0 -> 2
- net GND: track 84.1 -> 114.1 mm, vias 8 -> 13
- net /IMUSDA: track 20.1 -> 36.9 mm, vias 1 -> 4
- net /IMUSCL: track 17.3 -> 31.2 mm, vias 0 -> 3
- net /M2INB: track 16.5 -> 9.00 mm, vias 2 -> 1
- net /M2INA: track 88.0 -> 94.9 mm, vias 3 -> 6
- net /M3INA: track 60.7 -> 67.3 mm
- net /ir/IR2: track 46.0 -> 52.0 mm, vias 1 -> 3
- net /M4INA: track 92.2 -> 86.9 mm, vias 1 -> 2
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