File: lightweight/electrical design/layer3/layer3.kicad_sch (KiCad schematic)
At the start: 21 parts, among them J13 SH1.0 5P, J14 SH1.0 2P, J2 SH1.0 5P, J5 Conn_01x16_Socket, SW1 SW_SPDT, U1 TEENSY 4.0, U2 MOUDLE-SEEEDUINO-XIAO-ESP32C3, U4 74LVC2G04, U5 74LVC2G04, U6 74LVC2G04

Commit message: update lw l3 pcb
Parts:
- removed J14: SH1.0 2P, Connector_JST:JST_SH_SM02B-SRSS-TB_1x02-1MP_P1.00mm_Horizontal, symbol Connector:Conn_01x02_Pin
- removed U3: ~, libraries:OpenMV H7 R2, symbol Device:OpenMV_H7_R2
- added J5: Conn_01x03_Pin, Connector_JST:JST_XH_B3B-XH-A_1x03_P2.50mm_Vertical, symbol Connector:Conn_01x03_Pin
- renumbered J5 to U3
Connections:
- net GNDD is gone; now on net GND: DRIBBLERJ2.3 (Pin_3), J13.2 (Pin_2), R5.1, U1.G1, U1.G3, U2.13 (GND), U5.2 (GND), U6.2 (GND)
- net +3V3: now also J5.2 (Pin_2)
- net +5V: now also J5.1 (Pin_1)
- net GND: now also J5.3 (Pin_3)
- net M1CS: no longer names the net of J2.4 (Pin_4)
- net M2CS: no longer names the net of J2.4 (Pin_4)
- net M3CS: no longer names the net of J2.4 (Pin_4)
- net M4CS: no longer names the net of J2.4 (Pin_4)
