File: open/electrical design/layer3/layer3.kicad_pcb (KiCad board)
At the start: 2 copper layers, 150 x 137.9 mm, 42 parts, among them J1 SH1.0 5P, J10 SH1.0 2P, J11 SH1.0 5P, J12 XH2.54 2P, J2 SH1.0 5P, J3 SH1.0 5P, J4 SH1.0 5P, J5 XH2.54 5P, J6 CAMERA1, J7 CAMERA2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

Commit message: WE'RE FREE
Routing:
- net /BTTX: track 0.00 -> 91.4 mm
- net /BTRX: track 0.00 -> 81.1 mm
Changed lines of the file:
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@@
   (segment (start 65.25 152.25) (end 48 135) (width 0.25) (layer "B.Cu") (net 72))
   (segment (start 48 125.59) (end 54.62 118.97) (width 0.25) (layer "B.Cu") (net 72))
+  (segment (start 122.62 157.25) (end 146.75 157.25) (width 0.25) (layer "B.Cu") (net 73))
+  (segment (start 146.75 157.25) (end 172 132) (width 0.25) (layer "B.Cu") (net 73))
+  (segment (start 172 112.73) (end 170.62 111.35) (width 0.25) (layer "B.Cu") (net 73))
+  (segment (start 172 132) (end 172 112.73) (width 0.25) (layer "B.Cu") (net 73))
+  (segment (start 108.455 156.175) (end 145.825 156.175) (width 0.25) (layer "B.Cu") (net 74))
+  (segment (start 145.825 156.175) (end 169 133) (width 0.25) (layer "B.Cu") (net 74))
+  (segment (start 107.38 157.25) (end 108.455 156.175) (width 0.25) (layer "B.Cu") (net 74))
+  (segment (start 169 115.51) (end 170.62 113.89) (width 0.25) (layer "B.Cu") (net 74))
+  (segment (start 169 133) (end 169 115.51) (width 0.25) (layer "B.Cu") (net 74))
   (via (at 119.75 153.5) (size 0.8) (drill 0.4) (layers "F.Cu" "B.Cu") (free) (net 75))
   (via (at 146 136.5) (size 0.8) (drill 0.4) (layers "F.Cu" "B.Cu") (free) (net 75))
